File: MicroFLiC_DAC_power_supply_1_1.sch (KiCad schematic (older format))
At the start: 69 parts, among them P1 Socket_1x2, P2 Header_1x2, P3 Socket_2x4, U1 AP1117E50, U2 AP1117, U3 AP1117, U4 LM317, U5 LM317

Commit message: Updated part descriptions
Parts:
- C11, C12, C13, C14, C15: Note Optional 10 nF X7R ceramic capacitor -> Optional 10 nF 0603 X7R ceramic capacitor
- C25, C26, C27: Note 10μF/10V/3Ω ESR tantalum capacitor -> 10μF/10V/3Ω ESR case A tantalum capacitor
- C28, C29: Note 1μ/25V/6.6Ω ESR tantalum capacitor -> 1μ/25V/6.6Ω ESR case A tantalum capacitor
- D1, D2, D3: Note 10V Zener diode -> 10V SOD-323 Zener diode
- D4, D5: Note 27V Zener diode -> 27V SOD-323 Zener diode
- D6, D7, D8, D9: Note General small signal SOD-323 diode -> Small signal SOD-323 diode
Changed lines of the file:
@@
 F 9 "Mouser" H 2500 1600 60  0001 C CNN "Alt. Supplier"
 F 10 "80-C0805C103K5R" H 2500 1600 60  0001 C CNN "Alt. Order Code"
-F 11 "Optional 10 nF X7R ceramic capacitor" H 2500 1600 60  0001 C CNN "Note"
+F 11 "Optional 10 nF 0603 X7R ceramic capacitor" H 2500 1600 60  0001 C CNN "Note"
 	1    2500 1600
 	0    1    1    0
@@
 F 9 "Mouser" H 4700 1300 60  0001 C CNN "Alt. Supplier"
 F 10 "771-TDZ10J115" H 4700 1300 60  0001 C CNN "Alt. Order Code"
-F 11 "10V Zener diode" H 4700 1300 60  0001 C CNN "Note"
+F 11 "10V SOD-323 Zener diode" H 4700 1300 60  0001 C CNN "Note"
 	1    4700 1300
 	0    1    1    0
@@
 F 9 "Mouser" H 4700 6150 60  0001 C CNN "Alt. Supplier"
 F 10 "771-TDZ27J115" H 4700 6150 60  0001 C CNN "Alt. Order Code"
-F 11 "27V Zener diode" H 4700 6150 60  0001 C CNN "Note"
+F 11 "27V SOD-323 Zener diode" H 4700 6150 60  0001 C CNN "Note"
 	1    4700 6150
 	0    1    1    0
@@
 F 9 "Mouser" H 6100 1300 60  0001 C CNN "Alt. Supplier"
 F 10 "581-TAJA106K010" H 6100 1300 60  0001 C CNN "Alt. Order Code"
-F 11 "10μF/10V/3Ω ESR tantalum capacitor" H 6100 1300 60  0001 C CNN "Note"
+F 11 "10μF/10V/3Ω ESR case A tantalum capacitor" H 6100 1300 60  0001 C CNN "Note"
 	1    6100 1300
 	1    0    0    -1
@@
 F 9 "Mouser" H 6400 6350 60  0001 C CNN "Alt. Supplier"
 F 10 "74-TMCMA1E105MTRF" H 6400 6350 60  0001 C CNN "Alt. Order Code"
-F 11 "1μ/25V/6.6Ω ESR tantalum capacitor" H 6400 6350 60  0001 C CNN "Note"
+F 11 "1μ/25V/6.6Ω ESR case A tantalum capacitor" H 6400 6350 60  0001 C CNN "Note"
 	1    6400 6350
 	1    0    0    -1
@@
 F 9 "Mouser" H 2500 3050 60  0001 C CNN "Alt. Supplier"
 F 10 "80-C0805C103K5R" H 2500 3050 60  0001 C CNN "Alt. Order Code"
-F 11 "Optional 10 nF X7R ceramic capacitor" H 2500 3050 60  0001 C CNN "Note"
+F 11 "Optional 10 nF 0603 X7R ceramic capacitor" H 2500 3050 60  0001 C CNN "Note"
 	1    2500 3050
 	0    1    1    0
@@
 F 9 "Mouser" H 2500 4850 60  0001 C CNN "Alt. Supplier"
 F 10 "80-C0805C103K5R" H 2500 4850 60  0001 C CNN "Alt. Order Code"
-F 11 "Optional 10 nF X7R ceramic capacitor" H 2500 4850 60  0001 C CNN "Note"
+F 11 "Optional 10 nF 0603 X7R ceramic capacitor" H 2500 4850 60  0001 C CNN "Note"
 	1    2500 4850
 	0    1    1    0
@@
 F 9 "Mouser" H 2500 6450 60  0001 C CNN "Alt. Supplier"
 F 10 "80-C0805C103K5R" H 2500 6450 60  0001 C CNN "Alt. Order Code"
-F 11 "Optional 10 nF X7R ceramic capacitor" H 2500 6450 60  0001 C CNN "Note"
+F 11 "Optional 10 nF 0603 X7R ceramic capacitor" H 2500 6450 60  0001 C CNN "Note"
 	1    2500 6450
 	0    1    1    0
@@
 F 9 "Mouser" H 2500 8250 60  0001 C CNN "Alt. Supplier"
 F 10 "80-C0805C103K5R" H 2500 8250 60  0001 C CNN "Alt. Order Code"
-F 11 "Optional 10 nF X7R ceramic capacitor" H 2500 8250 60  0001 C CNN "Note"
+F 11 "Optional 10 nF 0603 X7R ceramic capacitor" H 2500 8250 60  0001 C CNN "Note"
 	1    2500 8250
 	0    1    1    0
@@
 F 9 "Mouser" H 4700 2750 60  0001 C CNN "Alt. Supplier"
 F 10 "771-TDZ10J115" H 4700 2750 60  0001 C CNN "Alt. Order Code"
-F 11 "10V Zener diode" H 4700 2750 60  0001 C CNN "Note"
+F 11 "10V SOD-323 Zener diode" H 4700 2750 60  0001 C CNN "Note"
 	1    4700 2750
 	0    1    1    0
@@
 F 9 "Mouser" H 4700 4550 60  0001 C CNN "Alt. Supplier"
 F 10 "771-TDZ10J115" H 4700 4550 60  0001 C CNN "Alt. Order Code"
-F 11 "10V Zener diode" H 4700 4550 60  0001 C CNN "Note"
+F 11 "10V SOD-323 Zener diode" H 4700 4550 60  0001 C CNN "Note"
 	1    4700 4550
 	0    1    1    0
@@
 F 9 "Mouser" H 4700 7950 60  0001 C CNN "Alt. Supplier"
 F 10 "771-TDZ27J115" H 4700 7950 60  0001 C CNN "Alt. Order Code"
-F 11 "27V Zener diode" H 4700 7950 60  0001 C CNN "Note"
+F 11 "27V SOD-323 Zener diode" H 4700 7950 60  0001 C CNN "Note"
 	1    4700 7950
 	0    1    1    0
@@
 F 9 "Mouser" H 6400 2950 60  0001 C CNN "Alt. Supplier"
 F 10 "581-TAJA106K010" H 6400 2950 60  0001 C CNN "Alt. Order Code"
-F 11 "10μF/10V/3Ω ESR tantalum capacitor" H 6400 2950 60  0001 C CNN "Note"
+F 11 "10μF/10V/3Ω ESR case A tantalum capacitor" H 6400 2950 60  0001 C CNN "Note"
 	1    6400 2950
 	1    0    0    -1
@@
 F 9 "Mouser" H 6400 4750 60  0001 C CNN "Alt. Supplier"
 F 10 "581-TAJA106K010" H 6400 4750 60  0001 C CNN "Alt. Order Code"
-F 11 "10μF/10V/3Ω ESR tantalum capacitor" H 6400 4750 60  0001 C CNN "Note"
+F 11 "10μF/10V/3Ω ESR case A tantalum capacitor" H 6400 4750 60  0001 C CNN "Note"
 	1    6400 4750
 	1    0    0    -1
@@
 F 9 "Mouser" H 6400 8150 60  0001 C CNN "Alt. Supplier"
 F 10 "74-TMCMA1E105MTRF" H 6400 8150 60  0001 C CNN "Alt. Order Code"
-F 11 "1μ/25V/6.6Ω ESR tantalum capacitor" H 6400 8150 60  0001 C CNN "Note"
+F 11 "1μ/25V/6.6Ω ESR case A tantalum capacitor" H 6400 8150 60  0001 C CNN "Note"
 	1    6400 8150
 	1    0    0    -1
@@
 F 9 "Mouser" H 5400 5500 60  0001 C CNN "Alt. Supplier"
 F 10 "512-1N4148WS" H 5400 5500 60  0001 C CNN "Alt. Order Code"
-F 11 "General small signal SOD-323 diode" H 5400 5500 60  0001 C CNN "Note"
+F 11 "Small signal SOD-323 diode" H 5400 5500 60  0001 C CNN "Note"
 	1    5400 5500
 	1    0    0    -1
@@
 F 9 "Mouser" H 6100 6050 60  0001 C CNN "Alt. Supplier"
 F 10 "512-1N4148WS" H 6100 6050 60  0001 C CNN "Alt. Order Code"
-F 11 "General small signal SOD-323 diode" H 6100 6050 60  0001 C CNN "Note"
+F 11 "Small signal SOD-323 diode" H 6100 6050 60  0001 C CNN "Note"
 	1    6100 6050
 	0    1    1    0
@@
 F 9 "Mouser" H 5400 7300 60  0001 C CNN "Alt. Supplier"
 F 10 "512-1N4148WS" H 5400 7300 60  0001 C CNN "Alt. Order Code"
-F 11 "General small signal SOD-323 diode" H 5400 7300 60  0001 C CNN "Note"
+F 11 "Small signal SOD-323 diode" H 5400 7300 60  0001 C CNN "Note"
 	1    5400 7300
 	1    0    0    -1
@@
 F 9 "Mouser" H 6100 7850 60  0001 C CNN "Alt. Supplier"
 F 10 "512-1N4148WS" H 6100 7850 60  0001 C CNN "Alt. Order Code"
-F 11 "General small signal SOD-323 diode" H 6100 7850 60  0001 C CNN "Note"
+F 11 "Small signal SOD-323 diode" H 6100 7850 60  0001 C CNN "Note"
 	1    6100 7850
 	0    1    1    0
