File: MicroFLiC_DAC_power_supply.sch (KiCad schematic (older format))
At the start: 69 parts, among them P1 Socket_1x2, P2 Header_1x2, P3 Socket_2x4, U1 AP1117E50, U2 AP1117, U3 AP1117, U4 LM317, U5 LM317

Commit message: Fixed capacitor and DC-DC converter descriptiions
Parts:
- C1, C10, C16, C17, C18, C2, C3, C4, C5, C6, C7, C8, C9: Note 4μ7/25V X5R 0805 ceramic capacitor -> 4.7μF/25V X5R 0805 ceramic capacitor
- C19, C20: Note 1μ/50V X5R 0805 ceramic capacitor -> 1μF/50V X5R 0805 ceramic capacitor
- C21, C22, C23, C24: Note 10μ/6.3V X5R 0805 ceramic capacitor -> 10μF/6.3V X5R 0805 ceramic capacitor
- C28, C29: Note 1μ/25V/6.6Ω ESR case A tantalum capacitor -> 1μF/25V/6.6Ω ESR case A tantalum capacitor
- DC1, DC2, DC3: Note 12V in 9V out 2W DC-DC converter -> 2W 12V to 9V DC-DC converter
- DC4, DC5: Note 12V in 24V out 2W DC-DC converter -> 2W 12V to 24V DC-DC converter
Changed lines of the file:
@@
 LIBS:valves
 LIBS:jakub
-LIBS:MicroFLiC_DAC_power_supply_1_1-cache
+LIBS:MicroFLiC_DAC_power_supply-cache
 EELAYER 25 0
 EELAYER END
@@
 F 9 "Mouser" H 2500 1050 60  0001 C CNN "Alt. Supplier"
 F 10 "580-NML1209SC" H 2500 1050 60  0001 C CNN "Alt. Order Code"
-F 11 "12V in 9V out 2W DC-DC converter" H 2500 1050 60  0001 C CNN "Note"
+F 11 "2W 12V to 9V DC-DC converter" H 2500 1050 60  0001 C CNN "Note"
 	1    2500 1050
 	1    0    0    -1
@@
 F 9 "Mouser" H 700 1200 60  0001 C CNN "Alt. Supplier"
 F 10 "81-GRM21BR61E475MA2L" H 700 1200 60  0001 C CNN "Alt. Order Code"
-F 11 "4μ7/25V X5R 0805 ceramic capacitor" H 700 1200 60  0001 C CNN "Note"
+F 11 "4.7μF/25V X5R 0805 ceramic capacitor" H 700 1200 60  0001 C CNN "Note"
 	1    700  1200
 	1    0    0    -1
@@
 F 9 "Mouser" H 4200 6150 60  0001 C CNN "Alt. Supplier"
 F 10 "81-GRM219R61H105KA3D" H 4200 6150 60  0001 C CNN "Alt. Order Code"
-F 11 "1μ/50V X5R 0805 ceramic capacitor" H 4200 6150 60  0001 C CNN "Note"
+F 11 "1μF/50V X5R 0805 ceramic capacitor" H 4200 6150 60  0001 C CNN "Note"
 	1    4200 6150
 	1    0    0    -1
@@
 F 9 "Mouser" H 2500 5900 60  0001 C CNN "Alt. Supplier"
 F 10 "81-NMG1224SC" H 2500 5900 60  0001 C CNN "Alt. Order Code"
-F 11 "12V in 24V out 2W DC-DC converter" H 2500 5900 60  0001 C CNN "Note"
+F 11 "2W 12V to 24V DC-DC converter" H 2500 5900 60  0001 C CNN "Note"
 	1    2500 5900
 	1    0    0    -1
@@
 F 9 "Mouser" H 700 2650 60  0001 C CNN "Alt. Supplier"
 F 10 "81-GRM21BR61E475MA2L" H 700 2650 60  0001 C CNN "Alt. Order Code"
-F 11 "4μ7/25V X5R 0805 ceramic capacitor" H 700 2650 60  0001 C CNN "Note"
+F 11 "4.7μF/25V X5R 0805 ceramic capacitor" H 700 2650 60  0001 C CNN "Note"
 	1    700  2650
 	1    0    0    -1
@@
 F 9 "Mouser" H 700 4450 60  0001 C CNN "Alt. Supplier"
 F 10 "81-GRM21BR61E475MA2L" H 700 4450 60  0001 C CNN "Alt. Order Code"
-F 11 "4μ7/25V X5R 0805 ceramic capacitor" H 700 4450 60  0001 C CNN "Note"
+F 11 "4.7μF/25V X5R 0805 ceramic capacitor" H 700 4450 60  0001 C CNN "Note"
 	1    700  4450
 	1    0    0    -1
@@
 F 9 "Mouser" H 700 6050 60  0001 C CNN "Alt. Supplier"
 F 10 "81-GRM21BR61E475MA2L" H 700 6050 60  0001 C CNN "Alt. Order Code"
-F 11 "4μ7/25V X5R 0805 ceramic capacitor" H 700 6050 60  0001 C CNN "Note"
+F 11 "4.7μF/25V X5R 0805 ceramic capacitor" H 700 6050 60  0001 C CNN "Note"
 	1    700  6050
 	1    0    0    -1
@@
 F 9 "Mouser" H 700 7850 60  0001 C CNN "Alt. Supplier"
 F 10 "81-GRM21BR61E475MA2L" H 700 7850 60  0001 C CNN "Alt. Order Code"
-F 11 "4μ7/25V X5R 0805 ceramic capacitor" H 700 7850 60  0001 C CNN "Note"
+F 11 "4.7μF/25V X5R 0805 ceramic capacitor" H 700 7850 60  0001 C CNN "Note"
 	1    700  7850
 	1    0    0    -1
@@
 F 9 "Mouser" H 4200 4550 60  0001 C CNN "Alt. Supplier"
 F 10 "81-GRM21BR61E475MA2L" H 4200 4550 60  0001 C CNN "Alt. Order Code"
-F 11 "4μ7/25V X5R 0805 ceramic capacitor" H 4200 4550 60  0001 C CNN "Note"
+F 11 "4.7μF/25V X5R 0805 ceramic capacitor" H 4200 4550 60  0001 C CNN "Note"
 	1    4200 4550
 	1    0    0    -1
@@
 F 9 "Mouser" H 4200 2750 60  0001 C CNN "Alt. Supplier"
 F 10 "81-GRM21BR61E475MA2L" H 4200 2750 60  0001 C CNN "Alt. Order Code"
-F 11 "4μ7/25V X5R 0805 ceramic capacitor" H 4200 2750 60  0001 C CNN "Note"
+F 11 "4.7μF/25V X5R 0805 ceramic capacitor" H 4200 2750 60  0001 C CNN "Note"
 	1    4200 2750
 	1    0    0    -1
@@
 F 9 "Mouser" H 4200 1300 60  0001 C CNN "Alt. Supplier"
 F 10 "81-GRM21BR61E475MA2L" H 4200 1300 60  0001 C CNN "Alt. Order Code"
-F 11 "4μ7/25V X5R 0805 ceramic capacitor" H 4200 1300 60  0001 C CNN "Note"
+F 11 "4.7μF/25V X5R 0805 ceramic capacitor" H 4200 1300 60  0001 C CNN "Note"
 	1    4200 1300
 	1    0    0    -1
@@
 F 9 "Mouser" H 4200 7950 60  0001 C CNN "Alt. Supplier"
 F 10 "81-GRM219R61H105KA3D" H 4200 7950 60  0001 C CNN "Alt. Order Code"
-F 11 "1μ/50V X5R 0805 ceramic capacitor" H 4200 7950 60  0001 C CNN "Note"
+F 11 "1μF/50V X5R 0805 ceramic capacitor" H 4200 7950 60  0001 C CNN "Note"
 	1    4200 7950
 	1    0    0    -1
@@
 F 9 "Mouser" H 1500 1200 60  0001 C CNN "Alt. Supplier"
 F 10 "81-GRM21BR61E475MA2L" H 1500 1200 60  0001 C CNN "Alt. Order Code"
-F 11 "4μ7/25V X5R 0805 ceramic capacitor" H 1500 1200 60  0001 C CNN "Note"
+F 11 "4.7μF/25V X5R 0805 ceramic capacitor" H 1500 1200 60  0001 C CNN "Note"
 	1    1500 1200
 	1    0    0    -1
@@
 F 9 "Mouser" H 1500 2650 60  0001 C CNN "Alt. Supplier"
 F 10 "81-GRM21BR61E475MA2L" H 1500 2650 60  0001 C CNN "Alt. Order Code"
-F 11 "4μ7/25V X5R 0805 ceramic capacitor" H 1500 2650 60  0001 C CNN "Note"
+F 11 "4.7μF/25V X5R 0805 ceramic capacitor" H 1500 2650 60  0001 C CNN "Note"
 	1    1500 2650
 	1    0    0    -1
@@
 F 9 "Mouser" H 1500 4450 60  0001 C CNN "Alt. Supplier"
 F 10 "81-GRM21BR61E475MA2L" H 1500 4450 60  0001 C CNN "Alt. Order Code"
-F 11 "4μ7/25V X5R 0805 ceramic capacitor" H 1500 4450 60  0001 C CNN "Note"
+F 11 "4.7μF/25V X5R 0805 ceramic capacitor" H 1500 4450 60  0001 C CNN "Note"
 	1    1500 4450
 	1    0    0    -1
@@
 F 9 "Mouser" H 1500 6050 60  0001 C CNN "Alt. Supplier"
 F 10 "81-GRM21BR61E475MA2L" H 1500 6050 60  0001 C CNN "Alt. Order Code"
-F 11 "4μ7/25V X5R 0805 ceramic capacitor" H 1500 6050 60  0001 C CNN "Note"
+F 11 "4.7μF/25V X5R 0805 ceramic capacitor" H 1500 6050 60  0001 C CNN "Note"
 	1    1500 6050
 	1    0    0    -1
@@
 F 9 "Mouser" H 1500 7850 60  0001 C CNN "Alt. Supplier"
 F 10 "81-GRM21BR61E475MA2L" H 1500 7850 60  0001 C CNN "Alt. Order Code"
-F 11 "4μ7/25V X5R 0805 ceramic capacitor" H 1500 7850 60  0001 C CNN "Note"
+F 11 "4.7μF/25V X5R 0805 ceramic capacitor" H 1500 7850 60  0001 C CNN "Note"
 	1    1500 7850
 	1    0    0    -1
@@
 F 9 "Mouser" H 6400 6350 60  0001 C CNN "Alt. Supplier"
 F 10 "74-TMCMA1E105MTRF" H 6400 6350 60  0001 C CNN "Alt. Order Code"
-F 11 "1μ/25V/6.6Ω ESR case A tantalum capacitor" H 6400 6350 60  0001 C CNN "Note"
+F 11 "1μF/25V/6.6Ω ESR case A tantalum capacitor" H 6400 6350 60  0001 C CNN "Note"
 	1    6400 6350
 	1    0    0    -1
@@
 F 9 "Mouser" H 2500 2500 60  0001 C CNN "Alt. Supplier"
 F 10 "580-NML1209SC" H 2500 2500 60  0001 C CNN "Alt. Order Code"
-F 11 "12V in 9V out 2W DC-DC converter" H 2500 2500 60  0001 C CNN "Note"
+F 11 "2W 12V to 9V DC-DC converter" H 2500 2500 60  0001 C CNN "Note"
 	1    2500 2500
 	1    0    0    -1
@@
 F 9 "Mouser" H 2500 4300 60  0001 C CNN "Alt. Supplier"
 F 10 "580-NML1209SC" H 2500 4300 60  0001 C CNN "Alt. Order Code"
-F 11 "12V in 9V out 2W DC-DC converter" H 2500 4300 60  0001 C CNN "Note"
+F 11 "2W 12V to 9V DC-DC converter" H 2500 4300 60  0001 C CNN "Note"
 	1    2500 4300
 	1    0    0    -1
@@
 F 9 "Mouser" H 2500 7700 60  0001 C CNN "Alt. Supplier"
 F 10 "81-NMG1224SC" H 2500 7700 60  0001 C CNN "Alt. Order Code"
-F 11 "12V in 24V out 2W DC-DC converter" H 2500 7700 60  0001 C CNN "Note"
+F 11 "2W 12V to 24V DC-DC converter" H 2500 7700 60  0001 C CNN "Note"
 	1    2500 7700
 	1    0    0    -1
@@
 F 9 "Mouser" H 6400 8150 60  0001 C CNN "Alt. Supplier"
 F 10 "74-TMCMA1E105MTRF" H 6400 8150 60  0001 C CNN "Alt. Order Code"
-F 11 "1μ/25V/6.6Ω ESR case A tantalum capacitor" H 6400 8150 60  0001 C CNN "Note"
+F 11 "1μF/25V/6.6Ω ESR case A tantalum capacitor" H 6400 8150 60  0001 C CNN "Note"
 	1    6400 8150
 	1    0    0    -1
@@
 F 9 "Mouser" H 5850 8350 60  0001 C CNN "Alt. Supplier"
 F 10 "581-08056D106MAT2A" H 5850 8350 60  0001 C CNN "Alt. Order Code"
-F 11 "10μ/6.3V X5R 0805 ceramic capacitor" H 5850 8350 60  0001 C CNN "Note"
+F 11 "10μF/6.3V X5R 0805 ceramic capacitor" H 5850 8350 60  0001 C CNN "Note"
 	1    5850 8350
 	1    0    0    -1
@@
 F 9 "Mouser" H 5850 6650 60  0001 C CNN "Alt. Supplier"
 F 10 "581-08056D106MAT2A" H 5850 6650 60  0001 C CNN "Alt. Order Code"
-F 11 "10μ/6.3V X5R 0805 ceramic capacitor" H 5850 6650 60  0001 C CNN "Note"
+F 11 "10μF/6.3V X5R 0805 ceramic capacitor" H 5850 6650 60  0001 C CNN "Note"
 	1    5850 6650
 	1    0    0    -1
@@
 F 9 "Mouser" H 5850 4950 60  0001 C CNN "Alt. Supplier"
 F 10 "581-08056D106MAT2A" H 5850 4950 60  0001 C CNN "Alt. Order Code"
-F 11 "10μ/6.3V X5R 0805 ceramic capacitor" H 5850 4950 60  0001 C CNN "Note"
+F 11 "10μF/6.3V X5R 0805 ceramic capacitor" H 5850 4950 60  0001 C CNN "Note"
 	1    5850 4950
 	1    0    0    -1
@@
 F 9 "Mouser" H 5850 3250 60  0001 C CNN "Alt. Supplier"
 F 10 "581-08056D106MAT2A" H 5850 3250 60  0001 C CNN "Alt. Order Code"
-F 11 "10μ/6.3V X5R 0805 ceramic capacitor" H 5850 3250 60  0001 C CNN "Note"
+F 11 "10μF/6.3V X5R 0805 ceramic capacitor" H 5850 3250 60  0001 C CNN "Note"
 	1    5850 3250
 	1    0    0    -1

Commit message: Fixed LDO feedback resistors and capacitors
Parts:
- C21, C22: value 10u/6.3V -> 4u7/25V; Alt. Order Code 581-08056D106MAT2A -> 81-GRM21BR61E475MA2L; Manufacturer Walsin -> Murata; Note 10μF/6.3V X5R 0805 ceramic capacitor -> 4.7μF/25V X5R 0805 ceramic capacitor; Order Code 2497051 -> 2362111; Part Number 0805X106K6R3CT -> GRM21BR61E475MA12L
- C23, C24: value 10u/6.3V -> 1u/50V; Alt. Order Code 581-08056D106MAT2A -> 81-GRM219R61H105KA3D; Manufacturer Walsin -> Murata; Note 10μF/6.3V X5R 0805 ceramic capacitor -> 1μF/50V X5R 0805 ceramic capacitor; Order Code 2497051 -> 1845750; Part Number 0805X106K6R3CT -> GRM219R61H105KA73D
- renumbered R5 to R1, R6 to R2, R7 to R3, R8 to R4, R1 to R5, R2 to R6, R3 to R7, R4 to R8
Other:
- moved on the sheet: R1, R2, R3, R4, R5, R6, R7, R8

Commit message: Fixed power output connector orientation
Changed lines of the file:
@@
 	1    0    0    -1
 $EndComp
+Text Label 5350 9000 0    60   ~ 0
+5V_GND
+Text Label 5350 9100 0    60   ~ 0
+-7.5V
+Text Label 5350 9200 0    60   ~ 0
+7.5V_GND
+Text Label 5350 9300 0    60   ~ 0
++7.5V
 Text Label 4350 9000 0    60   ~ 0
-5V_GND
++5V
 Text Label 4350 9100 0    60   ~ 0
--7.5V
+-19V
 Text Label 4350 9200 0    60   ~ 0
-7.5V_GND
+19V_GND
 Text Label 4350 9300 0    60   ~ 0
-+7.5V
-Text Label 5350 9000 0    60   ~ 0
-+5V
-Text Label 5350 9100 0    60   ~ 0
--19V
-Text Label 5350 9200 0    60   ~ 0
-19V_GND
-Text Label 5350 9300 0    60   ~ 0
 +19V
 Text Label 5650 8100 2    60   ~ 0
@@
 Connection ~ 3100 9100
 Wire Wire Line
-	4800 9000 4300 9000
-Wire Wire Line
-	4800 9100 4300 9100
-Wire Wire Line
-	4800 9200 4300 9200
-Wire Wire Line
-	4800 9300 4300 9300
+	5800 9000 5300 9000
+Wire Wire Line
+	5800 9100 5300 9100
+Wire Wire Line
+	5800 9200 5300 9200
+Wire Wire Line
+	5800 9300 5300 9300
 Wire Wire Line
 	5400 3650 5400 3400
@@
 Connection ~ 6400 3650
 Wire Wire Line
-	5800 9000 5300 9000
-Wire Wire Line
-	5800 9100 5300 9100
-Wire Wire Line
-	5800 9200 5300 9200
-Wire Wire Line
-	5800 9300 5300 9300
+	4800 9000 4300 9000
+Wire Wire Line
+	4800 9100 4300 9100
+Wire Wire Line
+	4800 9200 4300 9200
+Wire Wire Line
+	4800 9300 4300 9300
 Wire Wire Line
 	3200 2650 3200 3050

Commit message: Fixed connector descriptions
Parts:
- P1: value Socket_1x2 -> 1x2 socket strip
- P2: value Header_1x2 -> 1x2 header strip
- P3: value Socket_2x4 -> 2x4 socket strip
Changed lines of the file:
@@
 P 2700 9150
 F 0 "P1" H 2700 9300 50  0000 C CNN
-F 1 "Socket_1x2" V 2800 9150 50  0000 C CNN
+F 1 "1x2 socket strip" V 2800 9150 50  0000 C CNN
 F 2 "jakub:ESQ-102-33-G-S" H 2700 9150 60  0001 C CNN
 F 3 "" H 2700 9150 60  0000 C CNN
@@
 P 3500 9150
 F 0 "P2" H 3500 9300 50  0000 C CNN
-F 1 "Header_1x2" V 3600 9150 50  0000 C CNN
+F 1 "1x2 header strip" V 3600 9150 50  0000 C CNN
 F 2 "Pin_Headers:Pin_Header_Straight_1x02" H 3500 9150 60  0001 C CNN
 F 3 "" H 3500 9150 60  0000 C CNN
@@
 P 5050 9150
 F 0 "P3" H 5050 9400 50  0000 C CNN
-F 1 "Socket_2x4" H 5050 8900 50  0000 C CNN
+F 1 "2x4 socket strip" H 5050 8900 50  0000 C CNN
 F 2 "jakub:ESQ-104-33-G-D" H 5050 7950 60  0001 C CNN
 F 3 "" H 5050 7950 60  0000 C CNN

Commit message: Changed SOD-323 packages for larger pads.
Parts:
- D6, D7, D8, D9: footprint Diodes_SMD:SOD-323 -> jakub:SOD-323
Changed lines of the file:
@@
 F 0 "D6" H 5400 5600 50  0000 C CNN
 F 1 "1N4148" H 5400 5400 50  0000 C CNN
-F 2 "Diodes_SMD:SOD-323" H 5400 5500 50  0001 C CNN
+F 2 "jakub:SOD-323" H 5400 5500 50  0001 C CNN
 F 3 "" H 5400 5500 50  0000 C CNN
 F 4 "1N4148WS" H 5400 5500 60  0001 C CNN "Part Number"
@@
 F 0 "D8" H 6100 6150 50  0000 C CNN
 F 1 "1N4148" H 6100 5950 50  0000 C CNN
-F 2 "Diodes_SMD:SOD-323" H 6100 6050 50  0001 C CNN
+F 2 "jakub:SOD-323" H 6100 6050 50  0001 C CNN
 F 3 "" H 6100 6050 50  0000 C CNN
 F 4 "1N4148WS" H 6100 6050 60  0001 C CNN "Part Number"
@@
 F 0 "D7" H 5400 7400 50  0000 C CNN
 F 1 "1N4148" H 5400 7200 50  0000 C CNN
-F 2 "Diodes_SMD:SOD-323" H 5400 7300 50  0001 C CNN
+F 2 "jakub:SOD-323" H 5400 7300 50  0001 C CNN
 F 3 "" H 5400 7300 50  0000 C CNN
 F 4 "1N4148WS" H 5400 7300 60  0001 C CNN "Part Number"
@@
 F 0 "D9" H 6100 7950 50  0000 C CNN
 F 1 "1N4148" H 6100 7750 50  0000 C CNN
-F 2 "Diodes_SMD:SOD-323" H 6100 7850 50  0001 C CNN
+F 2 "jakub:SOD-323" H 6100 7850 50  0001 C CNN
 F 3 "" H 6100 7850 50  0000 C CNN
 F 4 "1N4148WS" H 6100 7850 60  0001 C CNN "Part Number"
